Commit message: parameterized model

File: urdf/clevon.urdf.xacro (robot description, xacro)
@@ -1,9 +1,13 @@
 <?xml version="1.0"?>
 <robot xmlns:xacro="http://www.ros.org/wiki/xacro" name="clevon">
+  <xacro:property name="cargobox_z_offset" value="0.338"/>
+  <xacro:property name="track_width" value="0.8"/>
+  <xacro:property name="wheel_base" value="1.74"/>
+  <xacro:property name="wheel_z_offset" value="0.148796"/>
   <link name="base_link">
     <visual>
-      <origin rpy="0 0 0" xyz="0 0 0"/>
+      <origin rpy="0 0 ${pi}" xyz="0 0 0"/>
       <geometry>
-        <mesh filename="package://clevon_description/meshes/702_with_cargobox_small.STL" scale="0.001 0.001 0.001"/>
+        <mesh filename="package://clevon_description/meshes/702_with_cargobox.STL" scale="0.001 0.001 0.001"/>
       </geometry>
       <material name="white">
@@ -12,6 +16,7 @@
     </visual>
     <collision>
+      <origin rpy="0 0 ${pi}" xyz="0 0 0"/>
       <geometry>
-        <mesh filename="package://clevon_description/meshes/702_with_cargobox_small.STL" scale="0.001 0.001 0.001"/>
+        <mesh filename="package://clevon_description/meshes/702_with_cargobox.STL" scale="0.001 0.001 0.001"/>
       </geometry>
     </collision>
@@ -19,7 +24,7 @@
   <link name="cargobox">
     <visual>
-      <origin rpy="0 0 0" xyz="0 0 0"/>
+      <origin rpy="0 0 ${pi}" xyz="0 0 0"/>
       <geometry>
-        <mesh filename="package://clevon_description/meshes/cargobox_v4.STL" scale="0.001 0.001 0.001"/>
+        <mesh filename="package://clevon_description/meshes/cargobox.STL" scale="0.001 0.001 0.001"/>
       </geometry>
       <material name="white">
@@ -28,97 +33,42 @@
     </visual>
     <collision>
+      <origin rpy="0 0 ${pi}" xyz="0 0 0"/>
       <geometry>
-        <mesh filename="package://clevon_description/meshes/cargobox_v4.STL" scale="0.001 0.001 0.001"/>
+        <mesh filename="package://clevon_description/meshes/cargobox.STL" scale="0.001 0.001 0.001"/>
       </geometry>
     </collision>
   </link>
-  <link name="wheel_1">
-    <visual>
-      <origin rpy="0 0 0" xyz="0 0 0"/>
-      <geometry>
-        <mesh filename="package://clevon_description/meshes/clevon_wheel.STL" scale="0.001 0.001 0.001"/>
-      </geometry>
-      <material name="black">
-        <color rgba="0 0 0 1" />
-      </material>
-    </visual>
-    <collision>
-      <geometry>
-        <mesh filename="package://clevon_description/meshes/clevon_wheel.STL" scale="0.001 0.001 0.001"/>
-      </geometry>
-    </collision>
-  </link>
-  <link name="wheel_2">
-    <visual>
-      <origin rpy="0 0 0" xyz="0 0 0"/>
-      <geometry>
-        <mesh filename="package://clevon_description/meshes/clevon_wheel.STL" scale="0.001 0.001 0.001"/>
-      </geometry>
-      <material name="black">
-        <color rgba="0 0 0 1" />
-      </material>
-    </visual>
-    <collision>
-      <geometry>
-        <mesh filename="package://clevon_description/meshes/clevon_wheel.STL" scale="0.001 0.001 0.001"/>
-      </geometry>
-    </collision>
-  </link>
-  <link name="wheel_3">
-    <visual>
-      <origin rpy="0 0 0" xyz="0 0 0"/>
-      <geometry>
-        <mesh filename="package://clevon_description/meshes/clevon_wheel.STL" scale="0.001 0.001 0.001"/>
-      </geometry>
-      <material name="black">
-        <color rgba="0 0 0 1" />
-      </material>
-    </visual>
-    <collision>
-      <geometry>
-        <mesh filename="package://clevon_description/meshes/clevon_wheel.STL" scale="0.001 0.001 0.001"/>
-      </geometry>
-    </collision>
-  </link>
-  <link name="wheel_4">
-    <visual>
-      <origin rpy="0 0 0" xyz="0 0 0"/>
-      <geometry>
-        <mesh filename="package://clevon_description/meshes/clevon_wheel.STL" scale="0.001 0.001 0.001"/>
-      </geometry>
-      <material name="black">
-        <color rgba="0 0 0 1" />
-      </material>
-    </visual>
-    <collision>
-      <geometry>
-        <mesh filename="package://clevon_description/meshes/clevon_wheel.STL" scale="0.001 0.001 0.001"/>
-      </geometry>
-    </collision>
-  </link>
+  <xacro:macro name="wheel" params="wheel_name reflect_x reflect_y">
+    <link name="${wheel_name}">
+      <visual>
+        <origin rpy="${pi/2} 0 ${pi*(reflect_y+1)/2}" xyz="0 0 0"/>
+        <geometry>
+          <mesh filename="package://clevon_description/meshes/clevon_wheel.STL" scale="0.001 0.001 0.001"/>
+        </geometry>
+        <material name="black">
+          <color rgba="0 0 0 1" />
+        </material>
+      </visual>
+      <collision>
+        <origin rpy="0 0 ${pi}" xyz="0 0 0"/>
+        <geometry>
+          <mesh filename="package://clevon_description/meshes/clevon_wheel.STL" scale="0.001 0.001 0.001"/>
+        </geometry>
+      </collision>
+    </link>
+    <joint name="base_link_to_${wheel_name}" type="fixed">
+      <parent link="base_link"/>
+      <child link="${wheel_name}"/>
+      <origin xyz="${wheel_base/2*reflect_x} ${track_width/2*reflect_y} ${wheel_z_offset}" rpy="0 0 0"/>
+    </joint>
+  </xacro:macro>
+  <xacro:wheel wheel_name="wheel_left_front" reflect_x="1" reflect_y="1"/>
+  <xacro:wheel wheel_name="wheel_left_rear" reflect_x="-1" reflect_y="1"/>
+  <xacro:wheel wheel_name="wheel_right_front" reflect_x="1" reflect_y="-1"/>
+  <xacro:wheel wheel_name="wheel_right_rear" reflect_x="-1" reflect_y="-1"/>
   <joint name="base_link_to_cargobox" type="fixed">
     <parent link="base_link"/>
     <child link="cargobox"/>
-    <origin xyz="0.56 0.07 0.49" rpy="0 0 0"/>
-  </joint>
-  <joint name="base_link_to_wheel_1" type="fixed">
-    <parent link="base_link"/>
-    <child link="wheel_1"/>
-    <origin xyz="0.1 0.15 0" rpy="1.57 0 0"/>
-  </joint>
-  <joint name="base_link_to_wheel_2" type="fixed">
-    <parent link="base_link"/>
-    <child link="wheel_2"/>
-    <origin xyz="1.8 0.15 0" rpy="1.57 0 0"/>
-  </joint>
-  <joint name="base_link_to_wheel_3" type="fixed">
-    <parent link="base_link"/>
-    <child link="wheel_3"/>
-    <origin xyz="0.1 1.0 0.6" rpy="-1.57 0 0"/>
-  </joint>
-  <joint name="base_link_to_wheel_4" type="fixed">
-    <parent link="base_link"/>
-    <child link="wheel_4"/>
-    <origin xyz="1.8 1.0 0.6" rpy="-1.57 0 0"/>
+    <origin xyz="0 0 ${cargobox_z_offset}" rpy="0 0 0"/>
   </joint>
 </robot>
